File: ev-driver.sch (KiCad schematic (older format))
At the start: 12 parts, among them IC1_%X%1 MOC3042M, P1_%X%1 CONN_01X02, Q1_%X%1 BC237, Q2_%X%1 TRIAC_BTA2

Commit message: Pre-branch commit
Connections:
- wire segments 34 -> 38
Changed lines of the file:
@@
 Connection ~ 4200 4550
 Wire Wire Line
-	1700 3500 3400 3500
+	1500 3500 3400 3500
 Wire Wire Line
 	6300 4450 9900 4450
@@
 Wire Wire Line
 	5100 3500 4650 3500
-Text HLabel 1700 3500 0    60   Input ~ 0
-ctrl_input_%X%
-Text HLabel 1700 3600 0    60   Input ~ 0
-ctrl_input_common
 Wire Notes Line
 	10250 2400 10250 4600
@@
 Wire Wire Line
 	8200 4550 9900 4550
+Text GLabel 1500 3350 1    60   Input ~ 0
+ctrl_input_%X%
+Wire Wire Line
+	1500 3350 1500 3500
+Text GLabel 10450 3650 1    60   Input ~ 0
+load_output_p_%X%
+Wire Wire Line
+	10450 3700 10450 4150
+Wire Wire Line
+	10450 4150 9550 4150
+Wire Wire Line
+	9550 4150 9550 4450
+Connection ~ 9550 4450
 $EndSCHEMATC
